Commit message: move workspace to git folder and update every files

File: capstone_resources/urdf/kinect_camera.urdf.xacro (robot description, xacro)
@@ -32,5 +32,5 @@
       <origin xyz="0 0 0" rpy="0 0 0"/>
       <visual>
-        <origin xyz="0 0 0" rpy="0 0 ${M_PI/2}"/>
+        <origin xyz="0 0 0" rpy="0 0 0"/> <!--${M_PI/2}-->
         <geometry>
           <mesh filename="package://husky_description/meshes/accessories/kinect.dae" />
